File: WIFI Module v1.1/Wifi Schemati.brd (EAGLE design)
At the start: 78.6 x 45.8 mm, 25 parts, among them IC1 PIC24FVXXKA302-SP

Commit message: ITS ALIVE
Currently (Hardware) Working, smaller board. Rev. 1.1
Parts:
- moved R2 0.66 mm to (22.9, 9.68), flipped to the top, turned to 118.7 degrees
- moved POWER 0.65 mm to (36.1, -13.2)
- moved SPI 0.65 mm to (48.8, -13.2)
- moved UART 0.65 mm to (55.1, -13.2)
- moved WIFI 0.65 mm to (42.5, -13.2)
- renumbered CR1 to LD33V3, JP1 to URT_OUT, JP2 to ESP_FIRMWARE, S1 to DIP, SHORT_TO_RST to RST_SHORT, SV1 to PICKIT, SV2 to TO_CB, U$1 to HUG_TOM
Routing:
- net GND: track 91.4 -> 95.6 mm
- net N$11: track 4.30 -> 3.66 mm
Other:
- board text added: "Messiah EMMS 2019"
- board text added: "PW"
- board text added: "SPI"
- board text added: "URT"
- board text added: "WFI"

Commit message: Gerbers and DRC fixes
Routing:
- net MISO: track 26.9 -> 26.4 mm
Changed lines of the file:
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@@
 <?xml version="1.0" encoding="utf-8"?>
 <!DOCTYPE eagle SYSTEM "eagle.dtd">
-<eagle version="9.2.2">
+<eagle version="9.3.0">
 <drawing>
 <settings>
-<setting alwaysvectorfont="no"/>
+<setting alwaysvectorfont="yes"/>
 <setting verticaltext="up"/>
 </settings>
@@
 <layer number="25" name="tNames" color="7" fill="1" visible="yes" active="yes"/>
 <layer number="26" name="bNames" color="7" fill="1" visible="yes" active="yes"/>
-<layer number="27" name="tValues" color="7" fill="1" visible="no" active="yes"/>
-<layer number="28" name="bValues" color="7" fill="1" visible="no" active="yes"/>
+<layer number="27" name="tValues" color="7" fill="1" visible="yes" active="yes"/>
+<layer number="28" name="bValues" color="7" fill="1" visible="yes" active="yes"/>
 <layer number="29" name="tStop" color="7" fill="3" visible="no" active="yes"/>
 <layer number="30" name="bStop" color="7" fill="6" visible="no" active="yes"/>
@@
 <wire x1="42.3058" y1="10.76224375" x2="42.3058" y2="9.694096875" width="0.762" layer="16"/>
 <wire x1="42.3058" y1="9.694096875" x2="43.447453125" y2="8.55244375" width="0.762" layer="16"/>
-<wire x1="69.237584375" y1="-6.31415" x2="69.286503125" y2="-6.36306875" width="0.762" layer="16"/>
 <wire x1="69.286503125" y1="-6.36306875" x2="73.056134375" y2="-6.36306875" width="0.762" layer="16"/>
 <wire x1="73.056134375" y1="-6.36306875" x2="74.75845625" y2="-4.660746875" width="0.762" layer="16"/>
@@
 <contactref element="TO_CB" pad="5"/>
 <wire x1="65.1611625" y1="-7.395465625" x2="68.25410625" y2="-7.395465625" width="0.762" layer="16"/>
-<wire x1="68.25410625" y1="-7.395465625" x2="69.286503125" y2="-6.36306875" width="0.762" layer="16"/>
 <wire x1="72.7858" y1="-2.688090625" x2="74.75845625" y2="-4.660746875" width="0.762" layer="16"/>
 <wire x1="72.7858" y1="3.14224375" x2="72.7858" y2="-2.688090625" width="0.762" layer="16"/>
 <wire x1="32.2397125" y1="4.40740625" x2="34.8828375" y2="4.40740625" width="0.762" layer="16"/>
 <wire x1="34.8828375" y1="4.40740625" x2="38.08149375" y2="1.20875" width="0.762" layer="16"/>
+<wire x1="68.25410625" y1="-7.395465625" x2="69.286503125" y2="-6.36306875" width="0.762" layer="16"/>
 </signal>
 <signal name="SPI_LIGHT">
@@
 <wire x1="62.6258" y1="2.045471875" x2="59.612784375" y2="-0.96754375" width="0.762" layer="16"/>
 <wire x1="59.612784375" y1="-0.96754375" x2="59.612784375" y2="-6.193540625" width="0.762" layer="16"/>
-<wire x1="59.612784375" y1="-15.612871875" x2="60.027315625" y2="-16.027403125" width="0.762" layer="16"/>
 <wire x1="59.612784375" y1="-6.193540625" x2="59.612784375" y2="-15.612871875" width="0.762" layer="1"/>
 <contactref element="TO_CB" pad="1"/>
-<wire x1="59.612784375" y1="-15.612871875" x2="61.555378125" y2="-17.555465625" width="0.762" layer="16"/>
-<wire x1="61.555378125" y1="-17.555465625" x2="65.1611625" y2="-17.555465625" width="0.762" layer="16"/>
+<wire x1="65.1611625" y1="-17.555465625" x2="61.555378125" y2="-17.555465625" width="0.762" layer="16"/>
+<wire x1="61.555378125" y1="-17.555465625" x2="59.612784375" y2="-15.612871875" width="0.762" layer="16"/>
 </signal>
 <signal name="MOSI">
